File: Project1/Project1.kicad_sch (KiCad schematic)
At the start: 28 parts, among them J1 Conn_01x01, J2 Conn_01x01, J3 Conn_01x01, J4 Conn_01x01, J5 Conn_01x01, SW1 SW_DP3T, U1 LM324, U2 LM324, U3 NE555P

Commit message: hiiiiiiiiiiii
Parts:
- removed J1, J2, J3, J4, J5: Conn_01x01, Connector:Banana_Jack_1Pin, symbol Connector_Generic:Conn_01x01
- added J1: Conn_01x03_Female, Connector_PinHeader_2.54mm:PinHeader_1x03_P2.54mm_Vertical, symbol Connector:Conn_01x03_Female
- added J2: Conn_01x02_Male, Connector_PinHeader_2.54mm:PinHeader_1x02_P2.54mm_Vertical, symbol Connector:Conn_01x02_Male
- added SW2: SW_DPDT_x2, Connector_PinSocket_2.54mm:PinSocket_1x03_P2.54mm_Vertical, symbol Switch:SW_DPDT_x2
- added TP1: Square Wave, TestPoint:TestPoint_Keystone_5010-5014_Multipurpose, symbol Connector:TestPoint
- added TP2: Triangle Wave, TestPoint:TestPoint_Keystone_5010-5014_Multipurpose, symbol Connector:TestPoint
- added TP3: Sine Wave, TestPoint:TestPoint_Keystone_5010-5014_Multipurpose, symbol Connector:TestPoint
- added TP4: Output Decision, TestPoint:TestPoint_Keystone_5010-5014_Multipurpose, symbol Connector:TestPoint
- added TP5: weak triangle, TestPoint:TestPoint_Keystone_5010-5014_Multipurpose, symbol Connector:TestPoint
- added TP6: Amplitude Adjusted, TestPoint:TestPoint_Keystone_5010-5014_Multipurpose, symbol Connector:TestPoint
- added TP7: weak square, TestPoint:TestPoint_Keystone_5010-5014_Multipurpose, symbol Connector:TestPoint
- R1: value 2.5k -> 100k
- R3: value 2.5k -> 10k
- R4: value 2.5k -> 2.2k
- R5: value 250k -> 220k
- SW1: footprint Button_Switch_SMD:SW_SP3T_PCM13 -> Switches:SW_SP3T
- U1, U2: footprint Package_DIP:DIP-16_W7.62mm -> Package_DIP:DIP-14_W7.62mm_Socket_LongPads
Connections:
- net +6V: now also J1.3 (Pin_3)
- net -6V: now also J1.1 (Pin_1)
- net GND: now also J1.2 (Pin_2), J2.1 (Pin_1), SW2.3 (C)
- net output_waveform: now also J2.2 (Pin_2)
- net sine_wave: now also TP3.1
- net square_wave: now also TP1.1
- net square_wave_weak: now also TP7.1
- net triangle_wave: now also TP2.1
- net triangle_weak: now also TP5.1
- net at R10.2, RV2.2, U2.7: now also TP6.1
- net at R7.1: now also SW2.1 (A); no longer SW1.3
- new net: SW1.3, SW2.2 (B), TP4.1
- no-connect marks 7 -> 8
Other:
- note added: "On/Off"
- moved on the sheet: R7, SW1A

Commit message: added switches and pot
Parts:
- removed R3: 10k, Resistor_THT:R_Axial_DIN0207_L6.3mm_D2.5mm_P7.62mm_Horizontal, symbol Device:R_US
- removed SW1: SW_DP3T, Switches:SW_SP3T, symbol Switch:SW_DP3T
- added RV4: 10k, Potentiometer_THT:Potentiometer_Bourns_3386P_Vertical, symbol Device:R_Potentiometer_US
- added SW1, SW3: SW_DPDT_x2, Connector_PinSocket_2.54mm:PinSocket_1x03_P2.54mm_Vertical, symbol Switch:SW_DPDT_x2
Connections:
- net sine_wave: now also SW1.1 (A)
- net square_wave: now also SW3.3 (C)
- net triangle_wave: now also SW1.3 (C)
- net at SW2.2 (B), TP4.1: now also SW3.2 (B)
- net at C1.2, C3.2, R1.2: now also RV4.1
- net at R5.1, U1.13 (-): now also RV4.2
- new net: SW1.2 (B), SW3.1 (A)
Other:
- moved on the sheet: TP4

Commit message: redesigned board
Parts:
- removed RV4: 10k, Potentiometer_THT:Potentiometer_Bourns_3386P_Vertical, symbol Device:R_Potentiometer_US
- added H1, H2, H3, H4: MountingHole, MountingHole:MountingHole_5mm, symbol Mechanical:MountingHole
- added R3: 10k, Resistor_THT:R_Axial_DIN0207_L6.3mm_D2.5mm_P7.62mm_Horizontal, symbol Device:R
- J1: footprint Connector_PinHeader_2.54mm:PinHeader_1x03_P2.54mm_Vertical -> Connector_PinSocket_2.54mm:PinSocket_1x03_P2.54mm_Vertical
- J2: footprint Connector_PinHeader_2.54mm:PinHeader_1x02_P2.54mm_Vertical -> Connector_PinSocket_2.54mm:PinSocket_1x02_P2.54mm_Vertical
- RV1, RV2, RV3: footprint Potentiometer_THT:Potentiometer_Bourns_3386P_Vertical -> custom:Chomkypot
- U3: footprint Package_DIP:DIP-8_W7.62mm -> Package_DIP:DIP-8_W7.62mm_Socket_LongPads
Connections:
- net at C1.2, C3.2, R1.2: now also R3.1
- net at R5.1, U1.13 (-): now also R3.2
